Commit message: Add in manual inverse kinematic

File: src/d1.urdf (robot description, URDF)
Before this commit: robot d1_description, 9 links, 8 joints
Links:
- added link tcp_link
Joints:
- added joint tcp_joint: type fixed, parent Link6, child tcp_link, origin xyz=0 0 0.0706 rpy=0 -1.5708 -1.5708
